Commit message: Migrate Spot simulation to Jazzy and add wall demo

File: spot_description/models/spot/model.urdf (robot description, URDF)
Before this commit: robot spot, 20 links, 19 joints
Links:
- added link imu_link
- added link lidar_link
- added link thermal_camera_link
- link base_link: geometry collision mesh filename=package://spot_description/models/spot/meshes/body_collisio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; visual mesh filename=package://spot_description/models/spot/meshes/body.dae
- link front_left_hip: geometry collision mesh filename=package://spot_description/models/spot/meshes/front_left_hi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; visual mesh filename=package://spot_description/models/spot/meshes/front_left_hi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
- link front_left_lower_leg: geometry collision mesh filename=package://spot_description/models/spot/meshes/front_left_lo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 scale=-1.82 0.97 0.98; visual mesh filename=package://spot_description/models/spot/meshes/front_left_lo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
- link front_left_upper_leg: geometry collision mesh filename=package://spot_description/models/spot/meshes/front_left_up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; visual mesh filename=package://spot_description/models/spot/meshes/front_left_up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
- link front_right_hip: geometry collision mesh filename=package://spot_description/models/spot/meshes/front_right_h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; visual mesh filename=package://spot_description/models/spot/meshes/front_right_h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
- link front_right_lower_leg: geometry collision mesh filename=package://spot_description/models/spot/meshes/front_right_l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 scale=-1.82 0.97 0.98; visual mesh filename=package://spot_description/models/spot/meshes/front_right_l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
- link front_right_upper_leg: geometry collision mesh filename=package://spot_description/models/spot/meshes/front_right_u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; visual mesh filename=package://spot_description/models/spot/meshes/front_right_u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
- link rear_left_hip: geometry collision mesh filename=package://spot_description/models/spot/meshes/rear_left_hip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; visual mesh filename=package://spot_description/models/spot/meshes/rear_left_hip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
- link rear_left_lower_leg: geometry collision mesh filename=package://spot_description/models/spot/meshes/rear_left_low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 scale=-1.82 0.97 0.98; visual mesh filename=package://spot_description/models/spot/meshes/rear_left_low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
- link rear_left_upper_leg: geometry collision mesh filename=package://spot_description/models/spot/meshes/rear_left_upp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; visual mesh filename=package://spot_description/models/spot/meshes/rear_left_upp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
- link rear_right_hip: geometry collision mesh filename=package://spot_description/models/spot/meshes/rear_right_hi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; visual mesh filename=package://spot_description/models/spot/meshes/rear_right_hi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
- link rear_right_lower_leg: geometry collision mesh filename=package://spot_description/models/spot/meshes/rear_right_lo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 scale=-1.82 0.97 0.98; visual mesh filename=package://spot_description/models/spot/meshes/rear_right_lo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
- link rear_right_upper_leg: geometry collision mesh filename=package://spot_description/models/spot/meshes/rear_right_up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; visual mesh filename=package://spot_description/models/spot/meshes/rear_right_up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
Joints:
- added joint imu_joint: type fixed, parent base_link, child imu_link, origin xyz=0 0 0 rpy=0 0 0
- added joint lidar_joint: type fixed, parent base_link, child lidar_link, origin xyz=0.223 0 0.11635 rpy=0 0 0
- added joint thermal_camera_joint: type fixed, parent base_link, child thermal_camera_link, origin xyz=-0.223 0 0.333 rpy=0 0 0
